Commit message: [upgrade][JBL]ZERITH H1 PRO V4.2: 1.固定从动轮 2.相机视角修正

File: ZERITH_H1_PRO_URDF/urdf/ZR_H1PRO-1.2.00.H.V4.3_URDF_2025.12.02.urdf (robot description, URDF)
Before this commit: robot ZR_H1PRO-1.2.00.H.V4.2_URDF_2025.11.17, 35 links, 34 joints
Links:
- link body_pitch_link: geometry collision mesh filename=package://ZR_H1PRO-1.2.00.H.V4.3_URDF_2025.12.02/meshes/bod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; visual mesh filename=package://ZR_H1PRO-1.2.00.H.V4.3_URDF_2025.12.02/meshes/bod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
- link body_yaw_link: geometry collision mesh filename=package://ZR_H1PRO-1.2.00.H.V4.3_URDF_2025.12.02/meshes/bod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; visual mesh filename=package://ZR_H1PRO-1.2.00.H.V4.3_URDF_2025.12.02/meshes/bod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
- link daogui_link: geometry collision mesh filename=package://ZR_H1PRO-1.2.00.H.V4.3_URDF_2025.12.02/meshes/dao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; visual mesh filename=package://ZR_H1PRO-1.2.00.H.V4.3_URDF_2025.12.02/meshes/dao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
- link dipan_link: geometry collision mesh filename=package://ZR_H1PRO-1.2.00.H.V4.3_URDF_2025.12.02/meshes/dip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; visual mesh filename=package://ZR_H1PRO-1.2.00.H.V4.3_URDF_2025.12.02/meshes/dip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
- link left_elbow_link: geometry collision mesh filename=package://ZR_H1PRO-1.2.00.H.V4.3_URDF_2025.12.02/meshes/lef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; visual mesh filename=package://ZR_H1PRO-1.2.00.H.V4.3_URDF_2025.12.02/meshes/lef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
- link left_end_effector_link: geometry collision mesh filename=package://ZR_H1PRO-1.2.00.H.V4.3_URDF_2025.12.02/meshes/lef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; visual mesh filename=package://ZR_H1PRO-1.2.00.H.V4.3_URDF_2025.12.02/meshes/lef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
- link left_front_wheel_link: geometry collision mesh filename=package://ZR_H1PRO-1.2.00.H.V4.3_URDF_2025.12.02/meshes/lef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; visual mesh filename=package://ZR_H1PRO-1.2.00.H.V4.3_URDF_2025.12.02/meshes/lef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
- link left_jaw_camera_link: geometry collision mesh filename=package://ZR_H1PRO-1.2.00.H.V4.3_URDF_2025.12.02/meshes/lef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; visual mesh filename=package://ZR_H1PRO-1.2.00.H.V4.3_URDF_2025.12.02/meshes/lef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
- link left_jaw_left_finger_link: geometry collision mesh filename=package://ZR_H1PRO-1.2.00.H.V4.3_URDF_2025.12.02/meshes/lef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; visual mesh filename=package://ZR_H1PRO-1.2.00.H.V4.3_URDF_2025.12.02/meshes/lef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
- link left_jaw_right_finger_link: geometry collision mesh filename=package://ZR_H1PRO-1.2.00.H.V4.3_URDF_2025.12.02/meshes/lef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; visual mesh filename=package://ZR_H1PRO-1.2.00.H.V4.3_URDF_2025.12.02/meshes/lef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
- link left_middle_wheel_link: geometry collision mesh filename=package://ZR_H1PRO-1.2.00.H.V4.3_URDF_2025.12.02/meshes/lef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; visual mesh filename=package://ZR_H1PRO-1.2.00.H.V4.3_URDF_2025.12.02/meshes/lef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
- link left_rear_wheel_link: geometry collision mesh filename=package://ZR_H1PRO-1.2.00.H.V4.3_URDF_2025.12.02/meshes/lef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; visual mesh filename=package://ZR_H1PRO-1.2.00.H.V4.3_URDF_2025.12.02/meshes/lef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
- link left_shoulder_pitch_link: geometry collision mesh filename=package://ZR_H1PRO-1.2.00.H.V4.3_URDF_2025.12.02/meshes/lef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; visual mesh filename=package://ZR_H1PRO-1.2.00.H.V4.3_URDF_2025.12.02/meshes/lef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
- link left_shoulder_roll_link: geometry collision mesh filename=package://ZR_H1PRO-1.2.00.H.V4.3_URDF_2025.12.02/meshes/lef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; visual mesh filename=package://ZR_H1PRO-1.2.00.H.V4.3_URDF_2025.12.02/meshes/lef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
- link left_shoulder_yaw_link: geometry collision mesh filename=package://ZR_H1PRO-1.2.00.H.V4.3_URDF_2025.12.02/meshes/lef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; visual mesh filename=package://ZR_H1PRO-1.2.00.H.V4.3_URDF_2025.12.02/meshes/lef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
- link left_wrist_pitch_link: geometry collision mesh filename=package://ZR_H1PRO-1.2.00.H.V4.3_URDF_2025.12.02/meshes/lef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; visual mesh filename=package://ZR_H1PRO-1.2.00.H.V4.3_URDF_2025.12.02/meshes/lef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
- link left_wrist_roll_link: geometry collision mesh filename=package://ZR_H1PRO-1.2.00.H.V4.3_URDF_2025.12.02/meshes/lef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; visual mesh filename=package://ZR_H1PRO-1.2.00.H.V4.3_URDF_2025.12.02/meshes/lef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
- link left_wrist_yaw_link: geometry collision mesh filename=package://ZR_H1PRO-1.2.00.H.V4.3_URDF_2025.12.02/meshes/lef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; visual mesh filename=package://ZR_H1PRO-1.2.00.H.V4.3_URDF_2025.12.02/meshes/lef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
- link neck_camera_link: geometry collision mesh filename=package://ZR_H1PRO-1.2.00.H.V4.3_URDF_2025.12.02/meshes/nec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; visual mesh filename=package://ZR_H1PRO-1.2.00.H.V4.3_URDF_2025.12.02/meshes/nec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
- link neck_pitch_link: geometry collision mesh filename=package://ZR_H1PRO-1.2.00.H.V4.3_URDF_2025.12.02/meshes/nec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; visual mesh filename=package://ZR_H1PRO-1.2.00.H.V4.3_URDF_2025.12.02/meshes/nec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
- link neck_yaw_link: geometry collision mesh filename=package://ZR_H1PRO-1.2.00.H.V4.3_URDF_2025.12.02/meshes/nec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; visual mesh filename=package://ZR_H1PRO-1.2.00.H.V4.3_URDF_2025.12.02/meshes/nec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
- link right_elbow_link: geometry collision mesh filename=package://ZR_H1PRO-1.2.00.H.V4.3_URDF_2025.12.02/meshes/rig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; visual mesh filename=package://ZR_H1PRO-1.2.00.H.V4.3_URDF_2025.12.02/meshes/rig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
- link right_end_effector_link: geometry collision mesh filename=package://ZR_H1PRO-1.2.00.H.V4.3_URDF_2025.12.02/meshes/rig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; visual mesh filename=package://ZR_H1PRO-1.2.00.H.V4.3_URDF_2025.12.02/meshes/rig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
- link right_front_wheel_link: geometry collision mesh filename=package://ZR_H1PRO-1.2.00.H.V4.3_URDF_2025.12.02/meshes/rig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; visual mesh filename=package://ZR_H1PRO-1.2.00.H.V4.3_URDF_2025.12.02/meshes/rig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
- link right_jaw_camera_link: geometry collision mesh filename=package://ZR_H1PRO-1.2.00.H.V4.3_URDF_2025.12.02/meshes/rig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; visual mesh filename=package://ZR_H1PRO-1.2.00.H.V4.3_URDF_2025.12.02/meshes/rig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
- link right_jaw_left_finger_link: geometry collision mesh filename=package://ZR_H1PRO-1.2.00.H.V4.3_URDF_2025.12.02/meshes/rig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; visual mesh filename=package://ZR_H1PRO-1.2.00.H.V4.3_URDF_2025.12.02/meshes/rig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
- link right_jaw_right_finger_link: geometry collision mesh filename=package://ZR_H1PRO-1.2.00.H.V4.3_URDF_2025.12.02/meshes/rig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; visual mesh filename=package://ZR_H1PRO-1.2.00.H.V4.3_URDF_2025.12.02/meshes/rig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
- link right_middle_wheel_link: geometry collision mesh filename=package://ZR_H1PRO-1.2.00.H.V4.3_URDF_2025.12.02/meshes/rig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; visual mesh filename=package://ZR_H1PRO-1.2.00.H.V4.3_URDF_2025.12.02/meshes/rig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
- link right_rear_wheel_link: geometry collision mesh filename=package://ZR_H1PRO-1.2.00.H.V4.3_URDF_2025.12.02/meshes/rig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; visual mesh filename=package://ZR_H1PRO-1.2.00.H.V4.3_URDF_2025.12.02/meshes/rig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
- link right_shoulder_pitch_link: geometry collision mesh filename=package://ZR_H1PRO-1.2.00.H.V4.3_URDF_2025.12.02/meshes/rig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; visual mesh filename=package://ZR_H1PRO-1.2.00.H.V4.3_URDF_2025.12.02/meshes/rig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
- link right_shoulder_roll_link: geometry collision mesh filename=package://ZR_H1PRO-1.2.00.H.V4.3_URDF_2025.12.02/meshes/rig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; visual mesh filename=package://ZR_H1PRO-1.2.00.H.V4.3_URDF_2025.12.02/meshes/rig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
- link right_shoulder_yaw_link: geometry collision mesh filename=package://ZR_H1PRO-1.2.00.H.V4.3_URDF_2025.12.02/meshes/rig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; visual mesh filename=package://ZR_H1PRO-1.2.00.H.V4.3_URDF_2025.12.02/meshes/rig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
- link right_wrist_pitch_link: geometry collision mesh filename=package://ZR_H1PRO-1.2.00.H.V4.3_URDF_2025.12.02/meshes/rig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; visual mesh filename=package://ZR_H1PRO-1.2.00.H.V4.3_URDF_2025.12.02/meshes/rig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
- link right_wrist_roll_link: geometry collision mesh filename=package://ZR_H1PRO-1.2.00.H.V4.3_URDF_2025.12.02/meshes/rig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; visual mesh filename=package://ZR_H1PRO-1.2.00.H.V4.3_URDF_2025.12.02/meshes/rig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
- link right_wrist_yaw_link: geometry collision mesh filename=package://ZR_H1PRO-1.2.00.H.V4.3_URDF_2025.12.02/meshes/rig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; visual mesh filename=package://ZR_H1PRO-1.2.00.H.V4.3_URDF_2025.12.02/meshes/rig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
Joints:
- joint left_front_wheel_joint: axis 0 1 0 -> 0 0 0; type continuous -> fixed
- joint left_jaw_camera_joint: origin xyz=0.096166 0 0.065657 rpy=1.1345 0 -1.5708 -> xyz=0.11933 0.009 0.060373 rpy=-2.0071 0 -1.5708
- joint left_rear_wheel_joint: axis 0 1 0 -> 0 0 0; type continuous -> fixed
- joint neck_camera_joint: origin xyz=0.0682334995183438 0.0324999999999979 -0.0364770320265024 rpy=-1.78023593389281 0 -1.5707963267949 -> xyz=0.0675568573382885 0.0324999999999979 -0.0363332072227294 rpy=-1.78023593389281 0 -1.5707963267949
- joint right_front_wheel_joint: axis 0 1 0 -> 0 0 0; type continuous -> fixed
- joint right_jaw_camera_joint: origin xyz=0.096166 0 0.065657 rpy=1.1345 0 -1.5708 -> xyz=0.11933 0.0090006 0.060373 rpy=-2.0071 0 -1.5708
- joint right_middle_wheel_joint: axis 0 1 0 -> 0 -1 0
- joint right_rear_wheel_joint: axis 0 1 0 -> 0 0 0; type continuous -> fixed
